Commit message: cartographer config

File: turtlebot3_description/urdf/turtlebot3_waffle.urdf (robot description, URDF)
Before this commit: robot turtlebot3_waffle, 7 links, 6 joints
Links:
- removed link t265_link
- added link laser, mass 1.2; collision mesh filename=package://turtlebot3_description/meshes/base/hokuyo_ust10.s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 scale=0.01 0.01 0.01; visual mesh filename=package://turtlebot3_description/meshes/base/hokuyo_ust10.s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 scale=0.01 0.01 0.01
Joints:
- removed joint t265_joint 
- added joint scan_joint: type fixed, parent base_link, child laser, origin xyz=0.2 0 0.195722 rpy=0 0 3.14
